Commit message: added nodes

File: ros2_ws/src/robot_bringup/urdf/product.urdf (robot description, URDF)
Before this commit: robot product_box, 1 links, 0 joints
Links:
- removed link box_link
- added link box, mass 0.5; collision mesh filename=file://$(find ur5_robotiq_description)/meshes/products/prod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 scale=1 1 1; visual mesh filename=file://$(find ur5_robotiq_description)/meshes/products/prod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 scale=1 1 1

File: ros2_ws/src/ur5_robotiq_description/urdf/ur.ros2_control.xacro (robot description, xacro)
@@ -28,5 +28,6 @@
         </xacro:if>
         <xacro:if value="${sim_ignition}">
-          <plugin>ign_ros2_control/IgnitionSystem</plugin>
+          <!-- <plugin>ign_ros2_control/IgnitionSystem</plugin> -->
+          <plugin>gazebo_ros2_control/GazeboSystem</plugin>
         </xacro:if>
         <xacro:if value="${use_fake_hardware}">

File: ros2_ws/src/ur5_robotiq_description/urdf/ur5_2f85/ur5_ros2_control.xacro (robot description, xacro)
@@ -4,5 +4,6 @@
     <ros2_control name="IgnitionSystem" type="system">
       <hardware>
-          <plugin>ign_ros2_control/IgnitionSystem</plugin>
+          <!-- <plugin>ign_ros2_control/IgnitionSystem</plugin> -->
+          <plugin>gazebo_ros2_control/GazeboSystem</plugin>
       </hardware>
       <joint name="${tf_prefix}shoulder_pan_joint">

File: ros2_ws/src/ur5_robotiq_description/urdf/ur5_robotiq_ros2_control.xacro (robot description, xacro)
@@ -4,5 +4,6 @@
     <ros2_control name="${robot_name}" type="system">
       <hardware>
-          <plugin>ign_ros2_control/IgnitionSystem</plugin>
+          <!-- <plugin>ign_ros2_control/IgnitionSystem</plugin> -->
+          <plugin>gazebo_ros2_control/GazeboSystem</plugin>
       </hardware>
       <joint name="${prefix}joint_1">
