Commit message: added manipulator

File: ros2_ws/src/robot_bringup/urdf/camera.urdf.xacro (robot description, xacro)
@@ -1,38 +1,15 @@
 <?xml version="1.0"?>
-<robot xmlns:xacro="http://wiki.ros.org/xacro" name="$(arg name)">
-  <!-- Macro to add camera to UR5 end-effector -->
-  <xacro:macro name="add_camera" params="parent_link">
-    <!-- Extension rod link -->
-<link name="camera_mount_link">
-    <visual name="rod_visual">
-        <origin xyz="0 0 0.04" rpy="0 0 0"/>
-        <geometry>
-        <cylinder radius="0.01" length="0.12"/>
-      </geometry>
-      <material name="Grey">
-        <color rgba="0.4 0.4 0.4 1"/>
-      </material>
-    </visual>
-    <collision>
-      <origin xyz="0 0 0.04" rpy="0 0 0"/>
-      <geometry>
-        <cylinder radius="0.01" length="0.08"/>
-      </geometry>
-    </collision>
-    <inertial>
-      <mass value="0.05"/>
-      <origin xyz="0 0 0.04" rpy="0 0 0"/>
-      <inertia ixx="0.00001" ixy="0" ixz="0"
-               iyy="0.00001" iyz="0"
-               izz="0.00001"/>
-    </inertial>
-  </link>
-    <!-- Camera Link -->
-    <link name="camera_link">
-      <!-- Camera Body -->
-      <visual name="camera_body_visual">
+<robot xmlns:xacro="http://wiki.ros.org/xacro" name="camera">
+  <!-- Macro: Small compact side-mounted camera -->
+  <xacro:macro name="add_camera" params="parent_link:=wrist_3_link">
+    <!-- ===================== -->
+    <!-- Camera Body (Rounded Box) -->
+    <!-- ===================== -->
+    <link name="camera_body_link">
+      <visual>
+        <!-- Slightly rounded housing -->
         <origin xyz="0 0 0" rpy="0 0 0"/>
         <geometry>
-          <box size="0.06 0.04 0.04"/>
+          <box size="0.05 0.03 0.03"/>
         </geometry>
         <material name="DarkGray">
@@ -40,61 +17,94 @@
         </material>
       </visual>
-      <!-- Collision -->
-      <collision name="camera_collision">
-        <origin xyz="0 0 0" rpy="0 0 0"/>
+      <collision>
         <geometry>
-          <box size="0.06 0.04 0.04"/>
+          <box size="0.05 0.03 0.03"/>
         </geometry>
       </collision>
-      <!-- Inertial (approximate) -->
       <inertial>
+        <mass value="0.12"/>
         <origin xyz="0 0 0" rpy="0 0 0"/>
-        <mass value="0.2"/>
-        <inertia ixx="0.0001" ixy="0.0" ixz="0.0"
-                 iyy="0.0001" iyz="0.0"
-                 izz="0.0001"/>
+        <inertia
+          ixx="1e-4" iyy="1e-4" izz="1e-4"
+          ixy="0.0" ixz="0.0" iyz="0.0"/>
       </inertial>
-</link>
-<!-- In your robot's xacro file -->
-<gazebo reference="camera_link">
-    <sensor name="camera_sensor" type="camera">
-        <pose>0 0 0.03 0 0 0</pose>
-      <camera>
-        <horizontal_fov>1.047</horizontal_fov>
-        <image>
-          <width>640</width>
-          <height>480</height>
-          <format>R8G8B8</format>
-        </image>
-        <clip>
-          <near>0.1</near>
-          <far>100</far>
-        </clip>
-      </camera>
-      <always_on>1</always_on>
-      <update_rate>30.0</update_rate>
-      <visualize>true</visualize>
-      <plugin name="gazebo_ros_camera" filename="libgazebo_ros_camera.so">
-        <ros>
-          <namespace>/ur5</namespace>
-          <remapping>image_raw:=camera/image_raw</remapping>
-        </ros>
-        <camera_name>camera</camera_name>
-        <frame_name>camera_link</frame_name>
-      </plugin>
-    </sensor>
-  </gazebo>
-  <!-- Joint between end-effector and rod -->
-  <joint name="camera_mount_joint" type="fixed">
-    <parent link="${parent_link}"/>
-    <child link="camera_mount_link"/>
-    <origin xyz="0 0 0" rpy="0 ${pi} ${pi}"/>
-  </joint>
-  <!-- Now attach camera to top of rod -->
-  <joint name="camera_joint" type="fixed">
-    <parent link="camera_mount_link"/>
-    <child link="camera_link"/>
-    <origin xyz="0 0 0.10" rpy="0 0 0"/>
-  </joint>
+    </link>
+    <!-- ===================== -->
+    <!-- Lens (small cylinder) -->
+    <!-- ===================== -->
+    <link name="camera_lens_link">
+      <visual>
+        <origin xyz="0 0.2 0.01" rpy="0 ${-pi/4} 0"/>
+        <geometry>
+          <cylinder radius="0.007" length="0.01"/>
+        </geometry>
+        <material name="LensBlack">
+          <color rgba="0.02 0.02 0.02 1"/>
+        </material>
+      </visual>
+      <collision>
+        <geometry>
+          <cylinder radius="0.007" length="0.01"/>
+        </geometry>
+      </collision>
+      <inertial>
+        <mass value="0.02"/>
+        <origin xyz="0 0 0" rpy="0 0 0"/>
+        <inertia
+          ixx="0.003" iyy="0.003" izz="0.003"
+          ixy="0.0" ixz="0.0" iyz="0.0"/>
+      </inertial>
+    </link>
+    <!-- ===================== -->
+    <!-- Gazebo Camera Sensor -->
+    <!-- ===================== -->
+    <gazebo reference="camera_lens_link">
+      <sensor name="rgb_camera" type="camera">
+        <pose>0 0 0.0 0 0 0</pose>
+        <update_rate>30.0</update_rate> <!-- keep 60Hz or 90Hz if stable -->
+        <always_on>true</always_on>
+        <visualize>true</visualize>
+        <camera>
+          <horizontal_fov>1.047</horizontal_fov>
+          <image>
+            <width>640</width>
+            <height>480</height>
+            <format>R8G8B8</format>
+          </image>
+          <clip>
+            <near>0.03</near>
+            <far>15.0</far>
+          </clip>
+        </camera>
+        <!-- Correct placement for plugin configuration -->
+        <plugin name="gazebo_ros_camera" filename="libgazebo_ros_camera.so">
+          <ros>
+            <namespace>/ur5</namespace>
+            <remapping>image_raw:=camera/image_raw</remapping>
+          </ros>
+          <camera_name>tcp</camera_name>
+          <frame_name>camera_lens_link</frame_name>
+          <publish_rate>30.0</publish_rate>  <!-- inside plugin -->
+          <queue_size>1</queue_size>          <!-- inside plugin -->
+        </plugin>
+      </sensor>
+    </gazebo>
+    <!-- ===================== -->
+    <!-- Joints -->
+    <!-- ===================== -->
+    <!-- Mount bracket to wrist body -->
+    <joint name="camera_bracket_joint" type="fixed">
+      <parent link="${parent_link}"/>
+      <!-- offset to the side and slightly forward -->
+      <child link="camera_body_link"/>
+      <!-- <origin xyz="0.04 0.07 -0.07" rpy="0 ${-pi/2} 0"/> -->
+      <origin xyz="0 -0.04 -0.02" rpy="0 ${-pi/2} 0"/>
+    </joint>
+    <!-- Attach lens to front of camera body -->
+    <joint name="camera_lens_joint" type="fixed">
+      <parent link="camera_body_link"/>
+      <child link="camera_lens_link"/>
+      <origin xyz="0 0 0.02" rpy="0 0 0"/>
+    </joint>
   </xacro:macro>
 </robot>

File: ros2_ws/src/robotiq_description/urdf/2f_85.ros2_control.xacro (robot description, xacro)
@@ -1,75 +1,42 @@
 <?xml version="1.0"?>
-<robot xmlns:xacro="http://www.ros.org/wiki/xacro">
-    <xacro:macro name="robotiq_gripper_ros2_control" params="
-        prefix
-        sim_ignition:=true">
-        <ros2_control name="IgnitionSystem" type="system">
-            <!-- Plugins -->
-           <hardware>
-                <plugin>ign_ros2_control/IgnitionSystem</plugin>
-            </hardware>
-            <!-- Joint interfaces -->
-            <!-- With Ignition or Hardware, they handle mimic joints, so we only need this command interface activated -->
-            <joint name="${prefix}robotiq_85_left_knuckle_joint">
-                <command_interface name="position" />
-                <state_interface name="position">
-                    <param name="initial_value">0.7929</param>
-                </state_interface>
-                <state_interface name="velocity"/>
-            </joint>
-            <!-- When simulating we need to include the rest of the gripper joints -->
-            <joint name="${prefix}robotiq_85_right_knuckle_joint">
-                <param name="mimic">${prefix}robotiq_85_left_knuckle_joint</param>
-                <param name="multiplier">-1</param>
-                <xacro:unless value="${sim_ignition}">
-                    <command_interface name="position"/>
-                    <state_interface name="position"/>
-                    <state_interface name="velocity"/>
-                </xacro:unless>
-            </joint>
-            <joint name="${prefix}robotiq_85_left_inner_knuckle_joint">
-                <param name="mimic">${prefix}robotiq_85_left_knuckle_joint</param>
-                <param name="multiplier">1</param>
-                <xacro:unless value="${sim_ignition}">
-                    <command_interface name="position"/>
-                    <state_interface name="position"/>
-                    <state_interface name="velocity"/>
-                </xacro:unless>
-            </joint>
-            <joint name="${prefix}robotiq_85_right_inner_knuckle_joint">
-                <param name="mimic">${prefix}robotiq_85_left_knuckle_joint</param>
-                <param name="multiplier">-1</param>
-                <xacro:unless value="${sim_ignition}">
-                    <command_interface name="position"/>
-                    <state_interface name="position"/>
-                    <state_interface name="velocity"/>
-                </xacro:unless>
-            </joint>
-            <joint name="${prefix}robotiq_85_left_finger_tip_joint">
-                <param name="mimic">${prefix}robotiq_85_left_knuckle_joint</param>
-                <param name="multiplier">-1</param>
-                <xacro:unless value="${sim_ignition}">
-                    <command_interface name="position"/>
-                    <state_interface name="position"/>
-                    <state_interface name="velocity"/>
-                </xacro:unless>
-            </joint>
-            <joint name="${prefix}robotiq_85_right_finger_tip_joint">
-                <param name="mimic">${prefix}robotiq_85_left_knuckle_joint</param>
-                <param name="multiplier">1</param>
-                <xacro:unless value="${sim_ignition}">
-                    <command_interface name="position"/>
-                    <state_interface name="position"/>
-                    <state_interface name="velocity"/>
-                </xacro:unless>
-            </joint>
-        </ros2_control>
-    </xacro:macro>
-    <gazebo>
-        <plugin filename="ign_ros2_control-system" name="ign_ros2_control::IgnitionROS2ControlPlugin">
-            <robot_param>robot_description</robot_param>
-            <robot_param_node>robot_state_publisher</robot_param_node>
-            <parameters>$(find robotiq_description)/config/robotiq_2f85_controllers.yaml</parameters>
-        </plugin>
-    </gazebo>
+<robot xmlns:xacro="http://wiki.ros.org/xacro">
+  <!--
+    Robotiq 2F-85 ROS2 Control Configuration for Gazebo Classic
+    Compatible with: ROS2 Humble, gazebo_ros2_control, UR5 integration
+  -->
+  <xacro:macro name="robotiq_gripper_ros2_control" params="prefix">
+    <ros2_control name="${prefix}robotiq_gripper" type="system">
+      <hardware>
+        <!-- ✅ Gazebo Classic plugin, not Ignition -->
+        <plugin>gazebo_ros2_control/GazeboSystem</plugin>
+      </hardware>
+      <!-- ✅ Primary controllable joint -->
+      <joint name="${prefix}robotiq_85_left_knuckle_joint">
+        <command_interface name="position"/>
+        <state_interface name="position"/>
+        <state_interface name="velocity"/>
+      </joint>
+      <!-- ✅ Mimic joints (handled by Gazebo, so they don’t need command interfaces) -->
+      <joint name="${prefix}robotiq_85_right_knuckle_joint">
+        <param name="mimic">${prefix}robotiq_85_left_knuckle_joint</param>
+        <param name="multiplier">-1</param>
+      </joint>
+      <joint name="${prefix}robotiq_85_left_inner_knuckle_joint">
+        <param name="mimic">${prefix}robotiq_85_left_knuckle_joint</param>
+        <param name="multiplier">1</param>
+      </joint>
+      <joint name="${prefix}robotiq_85_right_inner_knuckle_joint">
+        <param name="mimic">${prefix}robotiq_85_left_knuckle_joint</param>
+        <param name="multiplier">-1</param>
+      </joint>
+      <joint name="${prefix}robotiq_85_left_finger_tip_joint">
+        <param name="mimic">${prefix}robotiq_85_left_knuckle_joint</param>
+        <param name="multiplier">-1</param>
+      </joint>
+      <joint name="${prefix}robotiq_85_right_finger_tip_joint">
+        <param name="mimic">${prefix}robotiq_85_left_knuckle_joint</param>
+        <param name="multiplier">1</param>
+      </joint>
+    </ros2_control>
+  </xacro:macro>
 </robot>

Commit message: added IBVS control

File: ros2_ws/src/robot_bringup/urdf/camera.urdf.xacro (robot description, xacro)
@@ -57,4 +57,25 @@
     </link>
     <!-- ===================== -->
+    <!-- Optical frame (REP-103) -->
+    <!-- x right, y down, z forward -->
+    <!-- ===================== -->
+    <link name="camera_optical_frame">
+      <inertial>
+        <mass value="0.0001"/>
+        <origin xyz="0 0 0" rpy="0 0 0"/>
+        <inertia
+          ixx="1e-6" iyy="1e-6" izz="1e-6"
+          ixy="0.0" ixz="0.0" iyz="0.0"/>
+      </inertial>
+    </link>
+    <joint name="camera_optical_joint" type="fixed">
+      <parent link="camera_lens_link"/>
+      <child link="camera_optical_frame"/>
+      <!-- Rotation from URDF link frame (x forward, y left, z up)
+           to optical frame (x right, y down, z forward)
+           R = Rz(pi/2) * Rx(-pi/2) → rpy = (-pi/2, 0, -pi/2) -->
+      <origin xyz="0 0 0" rpy="${-pi/2} 0 ${-pi/2}"/>
+    </joint>
+    <!-- ===================== -->
     <!-- Gazebo Camera Sensor -->
     <!-- ===================== -->

File: ros2_ws/src/robot_bringup/urdf/ur5_arm.urdf.xacro (robot description, xacro)
@@ -122,4 +122,6 @@
      <origin xyz="0 0 0.8" rpy="0 0 0" />          <!-- position robot in the world -->
    </xacro:ur_robot>
+  <!-- Velocity control (for IBVS / forward_velocity_controller) -->
+  <xacro:ur_arm_transmission prefix="" hw_interface="VelocityJointInterface"/>
    <!-- === Camera before the gripper === -->
     <xacro:add_camera parent_link="wrist_3_link"/>

File: ros2_ws/src/robot_bringup/urdf/ur_macro.xacro (robot description, xacro)
@@ -3,4 +3,5 @@
   <xacro:include filename="$(find ur_description)/urdf/inc/ur_transmissions.xacro" />
   <xacro:include filename="$(find ur_description)/urdf/inc/ur_common.xacro" />
+  <!-- transmission_hw_interface:=hardware_interface/PositionJointInterface -->
   <xacro:macro name="ur_robot" params="
     name
@@ -13,5 +14,5 @@
     visual_parameters_file
     generate_ros2_control_tag:=true
-    transmission_hw_interface:=hardware_interface/PositionJointInterface
+    transmission_hw_interface:=velocity
     safety_limits:=false
     safety_pos_margin:=0.15
@@ -53,5 +54,6 @@
     <xacro:if value="${generate_ros2_control_tag}">
       <!-- ros2 control include -->
-      <xacro:include filename="$(find ur_description)/urdf/ur.ros2_control.xacro" />
+      <!-- <xacro:include filename="$(find ur_description)/urdf/ur.ros2_control.xacro" /> -->
+    <xacro:include filename="$(find robot_bringup)/urdf/ur_ros2_control.xacro" />
       <!-- ros2 control instance -->
       <xacro:ur_ros2_control
