Commit message: added yolov5

File: ros2_ws/src/ur5_robotiq_description/urdf/ur5_2f85/ur5_macro.xacro (robot description, xacro)
@@ -88,4 +88,5 @@
     keep_alive_count:=2"
     >
+    <xacro:property name="arm_scale" value="1.20"/>
     <!-- Load configuration data from the provided .yaml files -->
     <xacro:read_model_data
@@ -361,5 +362,5 @@
       <parent link="${tf_prefix}upper_arm_link" />
       <child link="${tf_prefix}forearm_link" />
-      <origin xyz="${forearm_x} ${forearm_y} ${forearm_z}" rpy="${forearm_roll} ${forearm_pitch} ${forearm_yaw}" />
+      <origin xyz="${forearm_x} ${forearm_y} ${forearm_z * arm_scale}" rpy="${forearm_roll} ${forearm_pitch} ${forearm_yaw}" />
       <axis xyz="0 0 1" />
       <limit lower="${elbow_joint_lower_limit}" upper="${elbow_joint_upper_limit}"
